Commit message: done

File: body.urdf (robot description, URDF)
Before this commit: robot robot, 3 links, 2 joints
Joints:
- removed joint FrontLeg_BackLeg
- added joint BackLeg_Torso: type revolute, parent BackLeg, child Torso, origin xyz=0.5 0 1.0 rpy=0 0 0, axis 0 1 0, limit lower=-3.14159 upper=3.14159 effort=0.0 velocity=0.0
- joint Torso_FrontLeg: origin xyz=0.5 0 1.0 rpy=0 0 0 -> xyz=1 0 0 rpy=0 0 0
